File: ads1115.kicad_sch (KiCad schematic)
At the start: 20 parts, among them J38 ads1115, J39 SI5351, J40 IN_RF, J41 IN_RF, U4 ADS1115IDGS

Commit message: Update
Parts:
- removed C26, C27, C28: 100nf, Capacitor_SMD:C_0805_2012Metric, symbol Device:C
- removed C29: 100n, Capacitor_SMD:C_0603_1608Metric, symbol Device:C
- removed J38: ads1115, Connector_PinSocket_2.54mm:PinSocket_1x10_P2.54mm_Vertical, symbol Connector:Conn_01x10_Pin
- removed J39: SI5351, Connector_PinHeader_2.54mm:PinHeader_1x07_P2.54mm_Vertical, symbol Connector:Conn_01x07_Pin
- removed J40, J41: IN_RF, Connector_Coaxial:SMA_Samtec_SMA-J-P-X-ST-EM1_EdgeMount, symbol Connector:Conn_Coaxial
- removed R58, R60, R62, R64, R66, R67: 10K, Resistor_SMD:R_0603_1608Metric, symbol Device:R_US
- removed R59, R61, R63, R65: 1K, Resistor_SMD:R_0603_1608Metric, symbol Device:R_US
- removed R68: 10K, Resistor_SMD:R_0805_2012Metric, symbol Device:R_US
- removed U4: ADS1115IDGS, Package_SO:TSSOP-10_3x3mm_P0.5mm, symbol Analog_ADC:ADS1115IDGS
