File: pic_analogs.kicad_sch (KiCad schematic)
At the start: 24 parts, among them J1 VFWD, J2 IN_RF, J3 OUT_RF, J4 VREV

Commit message: Update
Other:
- note added: "VSWR Bridge for Arduino"
- note removed: "Electgpl - VSWR Bridge for Arduino"
