File: pic_analogs.kicad_pcb (KiCad board)
At the start: 2 copper layers, 99.1 x 98.4 mm, 242 parts, among them J1 VFWD, J10 USB_B_Mini, J11 term_, J12 term_, J13 term_, J14 term_, J15 term_, J16 term_, J17 term_, J18 term_, J19 term_, J2 IN_RF, J20 term_, J21 term_, J22 term_, J23 term_, J24 term_, J25 term_, J26 term_, J27 term_, J28 term_, J29 term_, J3 OUT_RF, J30 term_, J31 term_, J32 ICD, J33 Micro_SD_Card, J34 Raspberry_Pi_zero_2w, J35 USB_A, J36 OledSpiST1306, J37 OledSpiST7789, J38 ads1115, J39 SI5351, J4 VREV, J40 IN_RF, J41 IN_RF, J42 OledSpiST1306, J43 tp_ft232_, J44 tp_ft232_, J45 tp_ft232_, J46 tp_ft232_, J47 tp_ft232_, J48 tp_ft232_, J49 tp_ft232_, J5 pickit, J50 tp_ft232_, J51 tp_ft232_, J52 USB_B_Mini, J53 F32R-1A7H1-11024, J54 tp_epaper, J56 tp_epaper, J57 tp_epaper, J58 tp_epaper, J59 tp_epaper, Q1 PMOS, SW1 mclr, SW2 rb4, SW3 rb5, SW4 mclr, SW5 ra5, SW6 ra4, SW7 ra5, U2 LM1117DT-3.3, U3 PIC18F4550-IPT, U4 ADS1115IDGS, U5 MRF24J40MA, U6 FT232BM, U7 LM1117DT-3.3, U8 25LCxxx, Y1 Crystal_GND24_Small, Y2 6Mhz

Commit message: Update
Parts:
- removed C26, C27, C28: 100nf, Capacitor_SMD:C_0805_2012Metric
- removed C29: 100n, Capacitor_SMD:C_0603_1608Metric
- removed J38: ads1115, Connector_PinSocket_2.54mm:PinSocket_1x10_P2.54mm_Vertical
- removed J39: SI5351, Connector_PinHeader_2.54mm:PinHeader_1x07_P2.54mm_Vertical
- removed J40, J41: IN_RF, Connector_Coaxial:SMA_Samtec_SMA-J-P-X-ST-EM1_EdgeMount
- removed R50, R51, R55: 4K7, Resistor_SMD:R_0603_1608Metric
- removed R58, R60, R62, R64, R66, R67: 10K, Resistor_SMD:R_0603_1608Metric
- removed R59, R61, R63, R65: 1K, Resistor_SMD:R_0603_1608Metric
- removed R68: 10K, Resistor_SMD:R_0805_2012Metric
- removed U4: ADS1115IDGS, Package_SO:TSSOP-10_3x3mm_P0.5mm
- added D13: RX, Diode_SMD:D_0805_2012Metric, F.Cu at (126.6, 140.1)
- added D14: RX, Diode_SMD:D_0805_2012Metric, F.Cu at (123.6, 140.1)
- added J6: oled128x64, kiC:SSD1306_No_Mounting_whitout_Holes, F.Cu at (152.6, 142.1)
- added R100: 2k2, Resistor_SMD:R_0805_2012Metric, F.Cu at (126.6, 144.5)
- added R103: 2k2, Resistor_SMD:R_0805_2012Metric, F.Cu at (123.7, 144.5)
- added R97: 2k2, Resistor_SMD:R_0603_1608Metric, F.Cu at (169.0, 149.6)
- C20, C22, C42, C43, R101, R102, R104, R48, R49, R96, R98, R99, U8: moved to F.Cu
- C44, C45, C46, C47: footprint Capacitor_SMD:C_0603_1608Metric -> Capacitor_SMD:C_0805_2012Metric
- D10, D11, D12: footprint Diode_SMD:D_1206_3216Metric -> Diode_SMD:D_SOD-128
- R69, R70, R71, R72, R73, R74, R75: footprint Resistor_SMD:R_0603_1608Metric -> Resistor_SMD:R_0805_2012Metric
- moved C22 94.6 mm to (215.2, 142.7)
- moved C30 90.3 mm to (215.1, 146.1), turned to 90 degrees
- moved R75 86.0 mm to (215.5, 150.3), turned to -90 degrees
- moved J52 82.3 mm to (212.6, 166.6), turned to -90 degrees
- moved R82 80.1 mm to (200.7, 173.8), turned to 90 degrees
- moved R83 78.6 mm to (199.1, 173.6), turned to -90 degrees
- moved J44 78.4 mm to (195.7, 175.6), turned to -90 degrees
- moved J50 78.4 mm to (197.4, 175.5), turned to 90 degrees
- moved R73 77.9 mm to (215.4, 154.1), turned to -90 degrees
- moved C35 77.5 mm to (202.4, 170.2), turned to 90 degrees
- moved J45 76.9 mm to (194.0, 175.0), turned to -90 degrees
- moved J49 76.8 mm to (192.2, 175.4), turned to -90 degrees
- moved U5 76.6 mm to (203.0, 147.9), turned to 0 degrees
- moved R94 76.3 mm to (206.6, 165.3), turned to 0 degrees
- moved C34 76.1 mm to (200.7, 170.2), turned to 90 degrees
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Connections:
- J34 pad 3: SDA_OLED_RPI -> SDA_RPI
- J34 pad 5: SCL_OLED_RPI -> SCL_RPI
- J34 pad 56: /magnetics/mcu_pic/rpi/TV -> Net-(J34-TV)
- J34 pad 67: Net-(J34-CORE) -> /magnetics/mcu_pic/rpi/CORE_RPI
- J34 pad 71: Net-(J34-WL_ON) -> unconnected-(J34-WL_ON-Pad71)
- J34 pad 72: Net-(J34-BT_ON) -> unconnected-(J34-BT_ON-Pad72)
- J37 pad 3: /magnetics/mcu_pic/rpi/display_oled/SCKL_SST -> GPIO26
- J37 pad 4: /magnetics/mcu_pic/rpi/display_oled/SDIN -> GPIO19
- JP4 pad 1: SCL_OLED_RPI -> SCL_RPI
- JP6 pad 1: SDA_OLED_RPI -> SDA_RPI
- R92 pad 2: USB_D- -> USB_D+
- U6 pad 7: USB_D- -> USB_D+
- U6 pad 8: USB_D+ -> USB_D-
Routing:
- net +3V3: track 265.9 -> 15.2 mm, vias 9 -> 0
- net +5V: track 131.6 -> 5.81 mm, vias 3 -> 0
- net SCL_OLED_RPI: track 117.4 -> 0.00 mm, vias 3 -> 0
- net GND: track 488.4 -> 371.3 mm, vias 480 -> 274
- net SDA_OLED_RPI: track 107.7 -> 0.00 mm
- net TX_RPI: track 75.9 -> 0.00 mm, vias 2 -> 0
- net V+_USB: track 74.9 -> 0.00 mm, vias 1 -> 0
- net MEASURE_ADDR0: track 72.6 -> 0.00 mm, vias 3 -> 0
- net RX_RPI: track 66.1 -> 0.00 mm, vias 2 -> 0
- net /magnetics/mcu_pic/rpi/mrf24j40/MISO_mrf24j40: track 47.8 -> 0.00 mm, vias 1 -> 0
- net /magnetics/mcu_pic/rpi/mrf24j40/MOSI_mrf24j40: track 46.4 -> 0.00 mm, vias 1 -> 0
- net /magnetics/mcu_pic/rpi/mrf24j40/CE0_mrf24j40: track 45.3 -> 0.00 mm, vias 1 -> 0
- net /magnetics/mcu_pic/rpi/mrf24j40/SCLK_mrf24j40: track 41.8 -> 0.00 mm, vias 1 -> 0
- net SCLK: track 40.3 -> 0.00 mm, vias 1 -> 0
- net MOSI: track 42.4 -> 3.16 mm, vias 1 -> 0
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
Commit message: Update
Parts:
- added J7: oled128x64, kiC:SSD1306_No_Mounting_whitout_Holes, F.Cu at (212.2, 129.3)
- moved J5 0.37 mm to (199.0, 132.4)
Routing:
- net SCL/SCK: track 67.4 -> 78.3 mm, vias 2 -> 3
- net SDA/MISO: track 82.8 -> 89.9 mm, vias 2 -> 3
- net GND: track 371.3 -> 374.1 mm
- net +3.3V: track 187.6 -> 190.1 mm
- net /magnetics/mcu_pic/pgd: track 34.0 -> 34.8 mm
- net /magnetics/mcu_pic/mclr: track 48.1 -> 47.4 mm

Commit message: Update
Parts:
- removed C42: 100n, Capacitor_SMD:C_0603_1608Metric
- removed R101: 10K, Resistor_SMD:R_0603_1608Metric
- removed R102, R104: 2k2, Resistor_SMD:R_0603_1608Metric
- moved R99 4.34 mm to (175.3, 147.1), turned to 0 degrees
- moved R98 3.53 mm to (186.6, 145.0), turned to 90 degrees
- moved U8 3.25 mm to (181.5, 146.4)
- moved C43 2.55 mm to (181.8, 142.7)
- moved R96 2.02 mm to (175.3, 144.1)
Connections:
- U8 pad 2: MISO -> /magnetics/mcu_pic/rpi/mrf24j40/MISO_mrf24j40
- U8 pad 5: MOSI -> /magnetics/mcu_pic/rpi/mrf24j40/MOSI_mrf24j40
- U8 pad 6: SCLK -> /magnetics/mcu_pic/rpi/mrf24j40/SCLK_mrf24j40
Routing:
- net +3V3: track 15.2 -> 0.00 mm
- net Net-(U8-~{WP}): track 4.53 -> 0.00 mm
- net MOSI: track 3.16 -> 0.00 mm
- net MISO: track 2.26 -> 0.00 mm
- net CE1: track 2.10 -> 0.00 mm

Commit message: Update
Changed lines of the file:
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@@
 		)
 		(min_thickness 0.254)
-		(fill yes
+		(fill
 			(thermal_gap 0.508)
 			(thermal_bridge_width 0.508)
@@
 		)
 		(min_thickness 0.254)
-		(fill yes
+		(fill
 			(thermal_gap 0.508)
 			(thermal_bridge_width 0.508)
@@
 		)
 		(min_thickness 0.254)
-		(fill yes
+		(fill
 			(thermal_gap 0.508)
 			(thermal_bridge_width 0.508)
@@
 		)
 		(min_thickness 0.254)
-		(fill yes
+		(fill
 			(thermal_gap 0.508)
 			(thermal_bridge_width 0.508)
@@
 		)
 		(min_thickness 0.254)
-		(fill yes
+		(fill
 			(thermal_gap 0.508)
 			(thermal_bridge_width 0.508)
@@
 		)
 		(min_thickness 0.254)
-		(fill yes
+		(fill
 			(thermal_gap 0.508)
 			(thermal_bridge_width 0.508)
@@
 	)
 	(zone
+		(net "GND")
+		(layers "F.Cu" "B.Cu")
+		(hatch edge 0.5)
+		(priority 1)
+		(connect_pads yes
+			(clearance 0)
+		)
+		(min_thickness 0.25)
+		(fill
+			(thermal_gap 0.5)
+			(thermal_bridge_width 0.5)
+			(island_removal_mode 0)
+		)
+		(polygon
+			(pts
+				(xy 189.7888 78.680842) (xy 189.7888 128.778) (xy 118.11 128.778) (xy 118.11 175.457778) (xy 120.452222 177.8)
+				(xy 218.44 177.8) (xy 218.44 80.01) (xy 217.110842 78.680842)
+			)
+		)
+	)
+	(zone
 		(layer "F.Mask")
 		(hatch edge 0.5)
@@
 		)
 		(min_thickness 0.25)
-		(fill yes
+		(fill
 			(thermal_gap 0.5)
 			(thermal_bridge_width 0.5)
@@
 		)
 		(min_thickness 0.254)
-		(fill yes
+		(fill
 			(thermal_gap 0.508)
 			(thermal_bridge_width 0.508)
@@
 		)
 		(min_thickness 0.254)
-		(fill yes
+		(fill
 			(thermal_gap 0.508)
 			(thermal_bridge_width 0.508)
@@
 		)
 		(min_thickness 0.25)
-		(fill yes
+		(fill
 			(thermal_gap 0.5)
 			(thermal_bridge_width 0.5)

Commit message: add files .
Parts:
- removed J11, J16, J17, J18, J19, J20, J21, J22, J24, J25, J26, J27, J28, J29, J30: term_, Connector:connector_pin_smd_05
- removed J32: ICD, Connector_PinHeader_2.54mm:PinHeader_1x06_P2.54mm_Vertical_SMD
- removed J51: tp_ft232_, kiC:TestPoint_Pad_1.0x1.0mm
- removed JP4, JP6: jp, Jumper:SolderJumper-2_P1.3mm_Open_RoundedPad1.0x1.5mm
- added C55: 100nf, Capacitor_SMD:C_0805_2012Metric, F.Cu at (151.8, 163.5)
- added C56: 100nf, Capacitor_SMD:C_0805_2012Metric, F.Cu at (156.1, 157.0)
- added D15: LED, Diode_SMD:D_0805_2012Metric, F.Cu at (152.7, 167.1)
- added J8: TP, Connector_PinHeader_2.54mm:PinHeader_2x08_P2.54mm_Vertical, F.Cu at (215.2, 108.2)
- added JP11: NL, Jumper:SolderJumper-2_P1.3mm_Open_RoundedPad1.0x1.5mm, F.Cu at (149.2, 150.3)
- added JP12: NL, Jumper:SolderJumper-2_P1.3mm_Open_RoundedPad1.0x1.5mm, F.Cu at (152.7, 150.3)
- added L3: L, Inductor_SMD:L_Neosid_Ms42, B.Cu at (208.8, 87.2)
- added Q10: FDN306P, Package_TO_SOT_SMD:SOT-23W, F.Cu at (151.0, 159.4)
- added Q11: FDN306P, Package_TO_SOT_SMD:SOT-23W, F.Cu at (155.7, 160.2)
- added Q9: 2N7002, Package_TO_SOT_SMD:SOT-23, F.Cu at (160.2, 159.4)
- added R51: 10K, Resistor_SMD:R_0805_2012Metric, F.Cu at (152.2, 154.7)
- added R55: 10K, Resistor_SMD:R_0805_2012Metric, F.Cu at (155.6, 163.5)
- added R58: 10K, Resistor_SMD:R_0805_2012Metric, F.Cu at (163.1, 156.2)
- added R59: 10K, Resistor_SMD:R_0805_2012Metric, F.Cu at (155.9, 166.2)
- C10, C12: footprint Capacitor_SMD:C_0603_1608Metric -> Capacitor_SMD:C_1206_3216Metric
- C11, C9: value 100n -> 15p; footprint Capacitor_SMD:C_0603_1608Metric -> Capacitor_SMD:C_0805_2012Metric
- J12, J13, J14, J15: value term_ -> ~; footprint Connector:connector_pin_smd_05 -> kiC:connector_pin_smd_1mm; moved to B.Cu
- J23: value term_ -> TP_VCC; footprint Connector:connector_pin_smd_05 -> TestPoint:TestPoint_THTPad_1.0x1.0mm_Drill0.5mm
- J31: footprint Connector:connector_pin_smd_05 -> kiC:connector_pin_smd_1mm; moved to B.Cu
- L2: value L -> 100mh
- R20, R21, R25, R26, R27, R28, R29, R30, R31, R32, R33, R45, R80, R81: moved to B.Cu
- R34, R35, R36, R39: moved to F.Cu
- moved J23 93.7 mm to (153.1, 175.1)
- moved SW2 45.0 mm to (196.3, 132.4), turned to -90 degrees
- moved R28 38.8 mm to (197.6, 133.3), turned to 180 degrees
- moved R27 36.9 mm to (195.8, 131.6), turned to 180 degrees
- moved R25 36.9 mm to (196.4, 129.9), turned to 180 degrees
- moved J7 31.3 mm to (193.1, 104.4), turned to 90 degrees
- moved SW3 24.2 mm to (204.5, 132.4), turned to -90 degrees
- moved SW1 22.3 mm to (213.0, 132.4), turned to -90 degrees
- moved R35 21.8 mm to (197.1, 81.2), turned to 90 degrees
- moved D3 21.3 mm to (194.4, 82.8)
- moved D4 21.1 mm to (194.4, 80.6)
- moved R31 20.5 mm to (204.5, 128.9), turned to 180 degrees
- moved J5 20.2 mm to (193.1, 113.1), turned to 180 degrees
- moved R32 19.7 mm to (204.6, 130.5), turned to 0 degrees
- moved R23 17.0 mm to (197.7, 123.9)
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Connections:
- C44 pad 2: +5V -> /magnetics/mcu_pic/rpi/epaper/vcc_epaper_OUT
- C45 pad 2: +5V -> /magnetics/mcu_pic/rpi/epaper/vcc_epaper_OUT
- J10 pad 1: +5F -> Net-(J10-VBUS)
- J23 pad 1: /magnetics/mcu_pic/RD4 -> /magnetics/mcu_pic/rpi/epaper/vcc_epaper_OUT
- L2 pad 1: +5V -> /magnetics/mcu_pic/rpi/epaper/vcc_epaper_OUT
Routing:
- net GND: track 374.1 -> 0.00 mm, vias 274 -> 0
- net +3.3V: track 190.1 -> 0.00 mm, vias 10 -> 0
- net SDA/MISO: track 89.9 -> 0.00 mm, vias 3 -> 0
- net SCL/SCK: track 78.3 -> 0.00 mm, vias 3 -> 0
- net /RF: track 62.5 -> 0.00 mm
- net RX/MOSI: track 48.7 -> 0.00 mm, vias 2 -> 0
- net +5F: track 48.4 -> 0.00 mm, vias 2 -> 0
- net /magnetics/mcu_pic/mclr: track 47.4 -> 0.00 mm, vias 2 -> 0
- net CS: track 35.7 -> 0.00 mm, vias 2 -> 0
- net /magnetics/mcu_pic/pgd: track 34.8 -> 0.00 mm, vias 1 -> 0
- net /magnetics/mcu_pic/pgc: track 34.3 -> 0.00 mm, vias 1 -> 0
- net /magnetics/mcu_pic/RB4: track 26.8 -> 0.00 mm
- net Net-(J33-DAT1): track 21.0 -> 0.00 mm
- net /magnetics/mcu_pic/rpi/us_D+: track 18.4 -> 0.00 mm
- net /magnetics/mcu_pic/rpi/us_D-: track 17.7 -> 0.00 mm
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Other:
- copper layers 2 -> 4
- board text removed: "2 CS 5 SCK 3 MOSI GND 3v3 7 MISO"

Commit message: update files
Parts:
- moved J13 4.76 mm to (203.0, 105.2)
- moved J12 3.45 mm to (202.5, 103.8)
- moved R24 1.32 mm to (214.3, 104.3)
- moved R74 0.23 mm to (188.9, 153.5)
Routing:
- net +3V3: track 0.00 -> 226.8 mm, vias 0 -> 4
- net +3.3V: track 0.00 -> 215.0 mm, vias 0 -> 2
- net +5V: track 0.00 -> 114.4 mm, vias 0 -> 1
- net SDA/MISO: track 0.00 -> 113.5 mm, vias 0 -> 4
- net SCL/SCK: track 0.00 -> 107.8 mm, vias 0 -> 2
- net RUN_PI: track 0.00 -> 98.2 mm, vias 0 -> 1
- net V+_USB: track 0.00 -> 96.7 mm, vias 0 -> 4
- net /magnetics/mcu_pic/rpi/mrf24j40/CE0_mrf24j40: track 0.00 -> 82.7 mm, vias 0 -> 3
- net GPIO18: track 0.00 -> 70.9 mm, vias 0 -> 4
- net /magnetics/mcu_pic/pgd: track 0.00 -> 70.6 mm, vias 0 -> 3
- net /magnetics/mcu_pic/rpi/mrf24j40/MISO_mrf24j40: track 0.00 -> 70.4 mm, vias 0 -> 3
- net CSB: track 0.00 -> 69.6 mm, vias 0 -> 3
- net /magnetics/mcu_pic/rpi/tx_rpi: track 0.00 -> 68.6 mm, vias 0 -> 1
- net /magnetics/mcu_pic/rpi/epaper/vcc_epaper_OUT: track 0.00 -> 67.7 mm, vias 0 -> 1
- net RX/MOSI: track 0.00 -> 66.5 mm, vias 0 -> 4
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