File: SWR_meter.kicad_pcb (KiCad board)
At the start: 4 copper layers, 99.1 x 98.4 mm, 217 parts, among them J1 VFWD, J10 USB_B_Mini, J2 IN_RF, J23 TP_VCC, J3 OUT_RF, J31 term_, J33 Micro_SD_Card, J34 Raspberry_Pi_zero_2w, J35 USB_A, J36 OledSpiST1306, J37 OledSpiST7789, J4 VREV, J42 OledSpiST1306, J43 tp_ft232_, J44 tp_ft232_, J45 tp_ft232_, J46 tp_ft232_, J47 tp_ft232_, J48 tp_ft232_, J49 tp_ft232_, J5 pickit, J50 tp_ft232_, J52 USB_B_Mini, J53 F32R-1A7H1-11024, J54 tp_epaper, J56 tp_epaper, J57 tp_epaper, J58 tp_epaper, J59 tp_epaper, J6 oled128x64, J7 oled128x64, J8 TP, Q1 PMOS, Q10 FDN306P, Q11 FDN306P, Q9 2N7002, SW1 mclr, SW2 rb4, SW3 rb5, SW4 mclr, SW5 ra5, SW6 ra4, SW7 ra5, U2 LM1117DT-3.3, U3 PIC18F4550-IPT, U5 MRF24J40MA, U6 FT232BM, U7 LM1117DT-3.3, U8 25LCxxx, Y1 Crystal_GND24_Small, Y2 6Mhz

Commit message: Release v1.0.0: updated schematic and PCB files
Parts:
- U5: footprint Module:MODULE_MRF24J40MA -> kiC:MODULE_MRF24J40MA
- moved J53 1.52 mm to (168.3, 173.2)
Routing:
- net GND: track 10.5 -> 23.6 mm, vias 14 -> 136
- net +3V3: track 226.8 -> 232.2 mm
- net /magnetics/mcu_pic/rpi/epaper/CONTROL: track 27.4 -> 24.9 mm
- net GPIO18: track 70.9 -> 73.4 mm
- net /magnetics/mcu_pic/rpi/epaper/VDD: track 43.2 -> 40.9 mm
- net GPIO17: track 40.5 -> 38.4 mm
- net /magnetics/mcu_pic/rpi/epaper/VGL: track 22.4 -> 20.6 mm
- net /magnetics/mcu_pic/rpi/epaper/VDL: track 8.23 -> 6.49 mm
- net GPIO22: track 45.1 -> 43.4 mm
- net /magnetics/mcu_pic/rpi/epaper/VCOM: track 9.23 -> 7.61 mm
- net Net-(J58-Pin_1): track 4.80 -> 3.28 mm
- net /magnetics/mcu_pic/rpi/epaper/GDR: track 7.23 -> 5.71 mm
- net /magnetics/mcu_pic/rpi/epaper/RESE: track 16.8 -> 18.3 mm
- net Net-(J57-Pin_1): track 8.73 -> 7.21 mm
- net Net-(J59-Pin_1): track 12.8 -> 11.3 mm
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