File: SWR_meter.kicad_sch (KiCad schematic)
At the start: 24 parts, among them J1 VFWD, J2 IN_RF, J3 OUT_RF, J4 VREV

Commit message: Release v1.0.0: updated schematic and PCB files
Other:
- moved on the sheet: J3
