File: display_oled.kicad_sch (KiCad schematic)
At the start: 7 parts, among them J36 OledSpiST1306, J37 OledSpiST7789

Commit message: Update
Parts:
- added J6: oled128x64, kiC:SSD1306_No_Mounting_whitout_Holes, symbol Connector:Conn_01x04_Pin
Connections:
- net +3V3: now also J6.2 (Pin_2)
- net GND: now also J6.1 (Pin_1)
- net SCL_OLED_RPI: now also J6.3 (Pin_3)
- net SDA_OLED_RPI: now also J6.4 (Pin_4)
- net SCKL_SST renamed GPIO26
- net SDIN renamed GPIO19
