File: epaper.kicad_sch (KiCad schematic)
At the start: 26 parts, among them J53 F32R-1A7H1-11024, J54 tp_epaper, J56 tp_epaper, J57 tp_epaper, J58 tp_epaper, J59 tp_epaper, Q1 PMOS

Commit message: Update
Parts:
- C44, C45, C46, C47: footprint Capacitor_SMD:C_0603_1608Metric -> Capacitor_SMD:C_0805_2012Metric
- D10, D11, D12: footprint Diode_SMD:D_1206_3216Metric -> Diode_SMD:D_SOD-128

Commit message: add files .
Parts:
- removed JP4, JP6: jp, Jumper:SolderJumper-2_P1.3mm_Open_RoundedPad1.0x1.5mm, symbol Jumper:Jumper_2_Open
- added C55, C56: 100nf, Capacitor_SMD:C_0805_2012Metric, symbol Device:C
- added D15: LED, Diode_SMD:D_0805_2012Metric, symbol Device:LED
- added J23: TP_VCC, TestPoint:TestPoint_THTPad_1.0x1.0mm_Drill0.5mm, symbol Connector:Conn_01x01_Pin
- added JP11, JP12: NL, Jumper:SolderJumper-2_P1.3mm_Open_RoundedPad1.0x1.5mm, symbol Jumper:Jumper_2_Open
- added Q10, Q11: FDN306P, Package_TO_SOT_SMD:SOT-23W, symbol FDN306P:FDN306P
- added Q9: 2N7002, Package_TO_SOT_SMD:SOT-23, symbol Transistor_FET:2N7002
- added R51, R55, R58, R59: 10K, Resistor_SMD:R_0805_2012Metric, symbol Device:R_US
- L2: value L -> 100mh
Connections:
- net +5V: now also JP12.2 (B); no longer C44.2, C45.2, L2.1
- net GND: now also C55.2, C56.2, Q9.2 (S), R55.2, R59.2
- new net: Q10.1, Q11.2, Q9.3 (D)
- new net: D15.1 (K), R59.1
- new net +3V3: JP11.2 (B)
- new net CONTROL: Q11.1, Q9.1 (G), R51.1, R55.1, R58.2
- new net GPIO24: R58.1
- new net GPIO25: R51.2
- new net vcc_epaper_IN: C56.1, JP11.1 (A), JP12.1 (A), Q10.3, Q11.3
- new net vcc_epaper_OUT: C44.2, C45.2, C55.1, D15.2 (A), J23.1 (Pin_1), L2.1, Q10.2
