File: ft232.kicad_sch (KiCad schematic)
At the start: 40 parts, among them J43 tp_ft232_, J44 tp_ft232_, J45 tp_ft232_, J46 tp_ft232_, J47 tp_ft232_, J48 tp_ft232_, J49 tp_ft232_, J50 tp_ft232_, J51 tp_ft232_, J52 USB_B_Mini, U6 FT232BM, U7 LM1117DT-3.3, Y2 6Mhz

Commit message: add files .
Parts:
- removed J51: tp_ft232_, kiC:TestPoint_Pad_1.0x1.0mm, symbol Connector:Conn_01x01_Pin
Changed lines of the file:
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@@
 	)
 	(junction
-		(at 215.9 29.21)
-		(diameter 0)
-		(color 0 0 0 0)
-	)
-	(junction
 		(at 148.59 132.08)
 		(diameter 0)
@@
 	(wire
 		(pts
-			(xy 204.47 29.21) (xy 215.9 29.21)
-		)
-		(stroke
-			(width 0)
-			(type default)
-		)
-	)
-	(wire
-		(pts
 			(xy 27.94 66.04) (xy 40.64 66.04)
 		)
@@
 					(unit 1)
 				)
-			)
-		)
-	)
-	(symbol
-		(lib_id "Connector:Conn_01x01_Pin")
-		(at 199.39 29.21 0)
-		(mirror x)
-		(unit 1)
-		(body_style 1)
-		(exclude_from_sim no)
-		(in_bom yes)
-		(on_board yes)
-		(in_pos_files yes)
-		(dnp no)
-		(property "Reference" "J51"
-			(at 198.12 27.94 0)
-			(show_name no)
-			(do_not_autoplace no)
-			(effects
-				(font
-					(size 1.27 1.27)
-				)
-			)
-		)
-		(property "Value" "tp_ft232_"
-			(at 208.28 27.94 0)
-			(show_name no)
-			(do_not_autoplace no)
-			(effects
-				(font
-					(size 1.27 1.27)
-				)
-			)
-		)
-		(property "Footprint" "kiC:TestPoint_Pad_1.0x1.0mm"
-			(at 199.39 29.21 0)
-			(hide yes)
-			(show_name no)
-			(do_not_autoplace no)
-			(effects
-				(font
-					(size 1.27 1.27)
-				)
-			)
-		)
-		(property "Datasheet" ""
-			(at 199.39 29.21 0)
-			(hide yes)
-			(show_name no)
-			(do_not_autoplace no)
-			(effects
-				(font
-					(size 1.27 1.27)
-				)
-			)
-		)
-		(property "Description" ""
-			(at 199.39 29.21 0)
-			(show_name no)
-			(do_not_autoplace no)
-			(effects
-				(font
-					(size 1.27 1.27)
-				)
-			)
-		)
-		(pin "1"
-		)
-		(instances
-			(project "project_pi"
-				(path "/787baf38-3f0d-4343-8d8d-fd5be619bbb1/043d7997-457e-4619-a5b3-825bed78c0a6"
-					(reference "J?")
-					(unit 1)
-				)
-				(path "/787baf38-3f0d-4343-8d8d-fd5be619bbb1/b9fd0ca8-f7e7-4588-ad19-ad837ba6f041"
-					(reference "J?")
-					(unit 1)
-				)
-				(path "/787baf38-3f0d-4343-8d8d-fd5be619bbb1/f2931b9b-6fcc-4199-91d8-d06fd17cb974"
-					(reference "J?")
-					(unit 1)
-				)
-				(path "/787baf38-3f0d-4343-8d8d-fd5be619bbb1/b5d23a5d-5098-4708-9d84-8e554856594a/32a7254d-5557-4ccc-9a6b-7cf735213f61"
-					(reference "J?")
-					(unit 1)
-				)
-				(path "/787baf38-3f0d-4343-8d8d-fd5be619bbb1/b5d23a5d-5098-4708-9d84-8e554856594a/8cc3d87e-66d3-4bb3-be5f-abca356f4cca"
-					(reference "J?")
-					(unit 1)
-				)
-				(path "/787baf38-3f0d-4343-8d8d-fd5be619bbb1/b5d23a5d-5098-4708-9d84-8e554856594a/e3fc7fc0-eca8-4036-a3b0-cc543ef64249"
-					(reference "J?")
-					(unit 1)
-				)
-			)
-			(project "pic_analogs"
-				(path "/b399551b-4b97-4302-8921-d6009c0adde4/1d579dcc-e933-4401-b651-260801c00407/84ab4a69-ccf3-4ce1-bace-67b0704405a9/9dead999-4346-4391-b927-b533728301aa/bf831764-54a3-4e4e-a84a-fb9339c9ae35"
-					(reference "J51")
-					(unit 1)
-				)

Commit message: Release v1.0.0: updated schematic and PCB files
Connections:
- net GND: no longer J52.6 (Shield)
- no-connect marks 0 -> 2
Other:
- moved on the sheet: U6
