File: mcu_pic.kicad_sch (KiCad schematic)
At the start: 66 parts, among them J10 USB_B_Mini, J11 term_, J12 term_, J13 term_, J14 term_, J15 term_, J16 term_, J17 term_, J18 term_, J19 term_, J20 term_, J21 term_, J22 term_, J23 term_, J24 term_, J25 term_, J26 term_, J27 term_, J28 term_, J29 term_, J30 term_, J31 term_, J32 ICD, J5 pickit, SW1 mclr, SW2 rb4, SW3 rb5, U2 LM1117DT-3.3, U3 PIC18F4550-IPT, Y1 Crystal_GND24_Small

Commit message: Update
Other:
- removed sheet memory_spi
Changed lines of the file:
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@@
-	)
-	(sheet
-		(at 26.67 81.28)
-		(size 29.21 22.86)
-		(exclude_from_sim no)
-		(in_bom yes)
-		(on_board yes)
-		(dnp no)
-		(fields_autoplaced yes)
-		(stroke
-			(width 0.1524)
-			(type solid)
-		)
-		(fill
-			(color 0 0 0 0)
-		)
-		(property "Sheetname" "memory_spi"
-			(at 26.67 80.5684 0)
-			(show_name no)
-			(do_not_autoplace no)
-			(effects
-				(font
-					(size 1.27 1.27)
-				)
-				(justify left bottom)
-			)
-		)
-		(property "Sheetfile" "memory_spi.kicad_sch"
-			(at 26.67 104.7246 0)
-			(show_name no)
-			(do_not_autoplace no)
-			(effects
-				(font
-					(size 1.27 1.27)
-				)
-				(justify left top)
-			)
-		)
-		(instances
-			(project "pic_analogs"
-				(path "/b399551b-4b97-4302-8921-d6009c0adde4/1d579dcc-e933-4401-b651-260801c00407/84ab4a69-ccf3-4ce1-bace-67b0704405a9"
-					(page "12")
-				)
-			)
-		)
 	)
 	(sheet

Commit message: Update
Parts:
- J12, J13, J14, J15, J16, J17, J18, J19, J20, J21, J22, J23, J24, J25, J26, J27, J28, J29: value term_ -> (none); footprint Connector:connector_pin_smd_05 -> kiC:connector_pin_smd_1mm
Changed lines of the file:
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@@
 			)
 		)
-		(property "Value" "term_"
+		(property "Value" ""
 			(at 100.33 109.22 0)
 			(show_name no)
@@
 			)
 		)
-		(property "Footprint" "Connector:connector_pin_smd_05"
+		(property "Footprint" "kiC:connector_pin_smd_1mm"
 			(at 100.33 110.49 0)
 			(hide yes)
@@
 			)
 		)
-		(property "Value" "term_"
+		(property "Value" ""
 			(at 100.33 101.6 0)
 			(show_name no)
@@
 			)
 		)
-		(property "Footprint" "Connector:connector_pin_smd_05"
+		(property "Footprint" "kiC:connector_pin_smd_1mm"
 			(at 100.33 102.87 0)
 			(hide yes)
@@
 			)
 		)
-		(property "Value" "term_"
+		(property "Value" ""
 			(at 191.77 91.44 0)
 			(show_name no)
@@
 			)
 		)
-		(property "Footprint" "Connector:connector_pin_smd_05"
+		(property "Footprint" "kiC:connector_pin_smd_1mm"
 			(at 191.77 92.71 0)
 			(hide yes)
@@
 			)
 		)
-		(property "Value" "term_"
+		(property "Value" ""
 			(at 191.77 88.9 0)
 			(show_name no)
@@
 			)
 		)
-		(property "Footprint" "Connector:connector_pin_smd_05"
+		(property "Footprint" "kiC:connector_pin_smd_1mm"
 			(at 191.77 90.17 0)
 			(hide yes)
@@
 			)
 		)
-		(property "Value" "term_"
+		(property "Value" ""
 			(at 191.77 104.14 0)
 			(show_name no)
@@
 			)
 		)
-		(property "Footprint" "Connector:connector_pin_smd_05"
+		(property "Footprint" "kiC:connector_pin_smd_1mm"
 			(at 191.77 105.41 0)
 			(hide yes)
@@
 			)
 		)
-		(property "Value" "term_"
+		(property "Value" ""
 			(at 190.5 53.34 0)
 			(show_name no)
@@
 			)
 		)
-		(property "Footprint" "Connector:connector_pin_smd_05"
+		(property "Footprint" "kiC:connector_pin_smd_1mm"
 			(at 190.5 54.61 0)
 			(hide yes)
@@
 			)
 		)
-		(property "Value" "term_"
+		(property "Value" ""
 			(at 191.77 93.98 0)
 			(show_name no)
@@
 			)
 		)
-		(property "Footprint" "Connector:connector_pin_smd_05"
+		(property "Footprint" "kiC:connector_pin_smd_1mm"
 			(at 191.77 95.25 0)
 			(hide yes)
@@
 			)
 		)
-		(property "Value" "term_"
+		(property "Value" ""
 			(at 101.6 63.5 0)
 			(show_name no)
@@
 			)
 		)
-		(property "Footprint" "Connector:connector_pin_smd_05"
+		(property "Footprint" "kiC:connector_pin_smd_1mm"
 			(at 101.6 64.77 0)
 			(hide yes)
@@
 			)
 		)
-		(property "Value" "term_"
+		(property "Value" ""
 			(at 101.6 60.96 0)
 			(show_name no)
@@
 			)
 		)
-		(property "Footprint" "Connector:connector_pin_smd_05"
+		(property "Footprint" "kiC:connector_pin_smd_1mm"
 			(at 101.6 62.23 0)
 			(hide yes)
@@
 			)
 		)
-		(property "Value" "term_"
+		(property "Value" ""
 			(at 100.33 104.14 0)
 			(show_name no)
@@
 			)
 		)
-		(property "Footprint" "Connector:connector_pin_smd_05"
+		(property "Footprint" "kiC:connector_pin_smd_1mm"
 			(at 100.33 105.41 0)
 			(hide yes)
@@
 			)
 		)
-		(property "Value" "term_"
+		(property "Value" ""
 			(at 191.77 101.6 0)
 			(show_name no)
@@
 			)
 		)
-		(property "Footprint" "Connector:connector_pin_smd_05"
+		(property "Footprint" "kiC:connector_pin_smd_1mm"
 			(at 191.77 102.87 0)
 			(hide yes)
@@
 			)
 		)
-		(property "Value" "term_"
+		(property "Value" ""
 			(at 190.5 58.42 0)
 			(show_name no)
@@
 			)
 		)
-		(property "Footprint" "Connector:connector_pin_smd_05"
+		(property "Footprint" "kiC:connector_pin_smd_1mm"
 			(at 190.5 59.69 0)
 			(hide yes)
@@
 			)
 		)
-		(property "Value" "term_"
+		(property "Value" ""
 			(at 190.5 55.88 0)
 			(show_name no)
@@
 			)
 		)
-		(property "Footprint" "Connector:connector_pin_smd_05"
+		(property "Footprint" "kiC:connector_pin_smd_1mm"
 			(at 190.5 57.15 0)
 			(hide yes)
@@
 			)
 		)
-		(property "Value" "term_"
+		(property "Value" ""
 			(at 100.33 106.68 0)
 			(show_name no)
@@
 			)
 		)
-		(property "Footprint" "Connector:connector_pin_smd_05"
+		(property "Footprint" "kiC:connector_pin_smd_1mm"
 			(at 100.33 107.95 0)
 			(hide yes)
@@
 			)
 		)
-		(property "Value" "term_"
+		(property "Value" ""
 			(at 191.77 106.68 0)
 			(show_name no)
@@
 			)
 		)
-		(property "Footprint" "Connector:connector_pin_smd_05"
+		(property "Footprint" "kiC:connector_pin_smd_1mm"
 			(at 191.77 107.95 0)
 			(hide yes)
@@
 			)
 		)
-		(property "Value" "term_"
+		(property "Value" ""
 			(at 191.77 96.52 0)
 			(show_name no)
@@
 			)
 		)
-		(property "Footprint" "Connector:connector_pin_smd_05"
+		(property "Footprint" "kiC:connector_pin_smd_1mm"
 			(at 191.77 97.79 0)
 			(hide yes)
@@
 			)
 		)
-		(property "Value" "term_"
+		(property "Value" ""
 			(at 101.6 66.04 0)
 			(show_name no)
@@
 			)
 		)
-		(property "Footprint" "Connector:connector_pin_smd_05"
+		(property "Footprint" "kiC:connector_pin_smd_1mm"
 			(at 101.6 67.31 0)
 			(hide yes)
@@
 			)
 		)
-		(property "Value" "term_"
+		(property "Value" ""
 			(at 101.6 53.34 0)
 			(show_name no)
@@
 			)
 		)
-		(property "Footprint" "Connector:connector_pin_smd_05"
+		(property "Footprint" "kiC:connector_pin_smd_1mm"
 			(at 101.6 54.61 0)
 			(hide yes)

Commit message: add files .
Parts:
- removed J11, J30: term_, Connector:connector_pin_smd_05, symbol Connector:Conn_01x01_Pin
- removed J16, J17, J18, J19, J20, J21, J22, J23, J24, J25, J26, J27, J28, J29: (no value), kiC:connector_pin_smd_1mm, symbol Connector:Conn_01x01_Pin
- removed J32: ICD, Connector_PinHeader_2.54mm:PinHeader_1x06_P2.54mm_Vertical_SMD, symbol Connector:Conn_01x05_Pin
- added J8: TP, Connector_PinHeader_2.54mm:PinHeader_2x08_P2.54mm_Vertical, symbol Connector:Conn_01x14_Pin
- added L3: L, Inductor_SMD:L_Neosid_Ms42, symbol Device:L
- C10, C12: footprint Capacitor_SMD:C_0603_1608Metric -> Capacitor_SMD:C_1206_3216Metric
- C11, C9: value 100n -> 15p; footprint Capacitor_SMD:C_0603_1608Metric -> Capacitor_SMD:C_0805_2012Metric
- J31: footprint Connector:connector_pin_smd_05 -> kiC:connector_pin_smd_1mm
Connections:
- net +5F: now also L3.1; no longer J10.1 (VBUS)
- net RC0: now also J8.8 (Pin_8)
- net RC1: now also J8.9 (Pin_9)
- net RC2: now also J8.10 (Pin_10)
- net RD4: now also J8.14 (Pin_14)
- net RD5: now also J8.11 (Pin_11)
- net RD6: now also J8.13 (Pin_13)
- net RD7: now also J8.12 (Pin_12)
- net RE0: now also J8.1 (Pin_1)
- net RE1: now also J8.3 (Pin_3)
- net RE2: now also J8.2 (Pin_2)
- net ra0: now also J8.6 (Pin_6)
- net ra3: now also J8.7 (Pin_7)
- net ra4: now also J8.5 (Pin_5)
- net ra5: now also J8.4 (Pin_4)
- new net: J10.1 (VBUS), L3.2
Other:
- moved on the sheet: C10, C11, C12, C13, C14, C15, C16, C17, C18, C19, C9, D3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

Commit message: Release v1.0.0: updated schematic and PCB files
Connections:
- net GND: no longer J10.6 (Shield)
- no-connect marks 0 -> 3
Other:
- moved on the sheet: U2
