File: memory_spi.kicad_sch (KiCad schematic)
At the start: 9 parts, among them U8 25LCxxx

Commit message: Update
Parts:
- removed C42: 100n, Capacitor_SMD:C_0603_1608Metric, symbol Device:C
- removed R101: 10K, Resistor_SMD:R_0603_1608Metric, symbol Device:R_US
- removed R102, R104: 2k2, Resistor_SMD:R_0603_1608Metric, symbol Device:R_US
Connections:
- net CE1 renamed CS
