File: oled_mcu.kicad_sch (KiCad schematic)
At the start: 5 parts, among them J42 OledSpiST1306

Commit message: Update
Parts:
- added J7: oled128x64, kiC:SSD1306_No_Mounting_whitout_Holes, symbol Connector:Conn_01x04_Pin
Connections:
- net +3.3V: now also J7.2 (Pin_2)
- net GND: now also J7.1 (Pin_1)
- net SCL/SCK: now also J7.3 (Pin_3)
- net SDA/MISO: now also J7.4 (Pin_4)
