File: rpi.kicad_sch (KiCad schematic)
At the start: 16 parts, among them J34 Raspberry_Pi_zero_2w, J35 USB_A

Commit message: Update
Parts:
- removed R50, R51, R55: 4K7, Resistor_SMD:R_0603_1608Metric, symbol Device:R
- added D13, D14: RX, Diode_SMD:D_0805_2012Metric, symbol Device:LED_Small
- added R100, R103: 2k2, Resistor_SMD:R_0805_2012Metric, symbol Device:R_US
- added R97: 2k2, Resistor_SMD:R_0603_1608Metric, symbol Device:R_US
Connections:
- net CORE_RPI: now also J34.67 (CORE)
- net GND: now also R100.1, R103.1
- net PWM0: now also D13.1 (K)
- net PWM1: now also D14.1 (K)
- net TV: now also R97.1; no longer J34.56 (TV)
- new net: J34.56 (TV), R97.2
- new net: D13.2 (A), R100.2
- new net: D14.2 (A), R103.2
- no-connect marks 0 -> 11

Commit message: Release v1.0.0: updated schematic and PCB files
Other:
- removed sheet ads1115
